Commit message: Fixed to work with humble
Signed-off-by: Martin Hoang <hoangmrt@schaeffler.com>

File: models/rby1a/urdf/model_v1.2.urdf (robot description, URDF)
Before this commit: robot RBY1_A_v1.2, 32 links, 31 joints
Links:
- link base: geometry visual mesh filename=file:///home/martin/umanoid_ws/src/rby1-sdk/models/rby1a/ur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
- link ee_finger_l1: geometry visual mesh filename=file:///home/martin/umanoid_ws/src/rby1-sdk/models/rby1a/ur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
- link ee_finger_l2: geometry visual mesh filename=file:///home/martin/umanoid_ws/src/rby1-sdk/models/rby1a/ur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
- link ee_finger_r1: geometry visual mesh filename=file:///home/martin/umanoid_ws/src/rby1-sdk/models/rby1a/ur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
- link ee_finger_r2: geometry visual mesh filename=file:///home/martin/umanoid_ws/src/rby1-sdk/models/rby1a/ur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
- link ee_left: geometry visual mesh filename=file:///home/martin/umanoid_ws/src/rby1-sdk/models/rby1a/ur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
- link ee_right: geometry visual mesh filename=file:///home/martin/umanoid_ws/src/rby1-sdk/models/rby1a/ur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
- link link_head_0: geometry visual mesh filename=file:///home/martin/umanoid_ws/src/rby1-sdk/models/rby1a/ur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
- link link_head_1: geometry visual mesh filename=file:///home/martin/umanoid_ws/src/rby1-sdk/models/rby1a/ur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
- link link_head_2: geometry visual mesh filename=file:///home/martin/umanoid_ws/src/rby1-sdk/models/rby1a/ur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
- link link_left_arm_0: geometry collision cylinder length=0.0700 radius=0.075; visual mesh filename=file:///home/martin/umanoid_ws/src/rby1-sdk/models/rby1a/ur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
- link link_left_arm_1: geometry collision cylinder length=0.2000 radius=0.050; visual mesh filename=file:///home/martin/umanoid_ws/src/rby1-sdk/models/rby1a/ur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
- link link_left_arm_2: geometry collision cylinder length=0.080000 radius=0.05; visual mesh filename=file:///home/martin/umanoid_ws/src/rby1-sdk/models/rby1a/ur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
- link link_left_arm_3: geometry collision cylinder length=0.1150 radius=0.04; visual mesh filename=file:///home/martin/umanoid_ws/src/rby1-sdk/models/rby1a/ur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
- link link_left_arm_4: geometry collision cylinder length=0.095000 radius=0.035; visual mesh filename=file:///home/martin/umanoid_ws/src/rby1-sdk/models/rby1a/ur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
- link link_left_arm_5: geometry collision cylinder length=0.2213 radius=0.075; visual mesh filename=file:///home/martin/umanoid_ws/src/rby1-sdk/models/rby1a/ur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
- link link_left_arm_6: geometry visual mesh filename=file:///home/martin/umanoid_ws/src/rby1-sdk/models/rby1a/ur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
- link link_right_arm_0: geometry collision cylinder length=0.0700 radius=0.075; visual mesh filename=file:///home/martin/umanoid_ws/src/rby1-sdk/models/rby1a/ur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
- link link_right_arm_1: geometry collision cylinder length=0.2 radius=0.05; visual mesh filename=file:///home/martin/umanoid_ws/src/rby1-sdk/models/rby1a/ur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
- link link_right_arm_2: geometry collision cylinder length=0.080000 radius=0.05; visual mesh filename=file:///home/martin/umanoid_ws/src/rby1-sdk/models/rby1a/ur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
- link link_right_arm_3: geometry collision cylinder length=0.1150 radius=0.04; visual mesh filename=file:///home/martin/umanoid_ws/src/rby1-sdk/models/rby1a/ur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
- link link_right_arm_4: geometry collision cylinder length=0.095 radius=0.035; visual mesh filename=file:///home/martin/umanoid_ws/src/rby1-sdk/models/rby1a/ur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
- link link_right_arm_5: geometry collision cylinder length=0.2213 radius=0.075; visual mesh filename=file:///home/martin/umanoid_ws/src/rby1-sdk/models/rby1a/ur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
- link link_right_arm_6: geometry visual mesh filename=file:///home/martin/umanoid_ws/src/rby1-sdk/models/rby1a/ur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
- link link_torso_0: geometry collision cylinder length=0.230 radius=0.105; visual mesh filename=file:///home/martin/umanoid_ws/src/rby1-sdk/models/rby1a/ur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
- link link_torso_1: geometry collision cylinder length=0.220 radius=0.115; visual mesh filename=file:///home/martin/umanoid_ws/src/rby1-sdk/models/rby1a/ur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
- link link_torso_2: geometry collision cylinder length=0.1600 radius=0.095; visual mesh filename=file:///home/martin/umanoid_ws/src/rby1-sdk/models/rby1a/ur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
- link link_torso_3: geometry visual mesh filename=file:///home/martin/umanoid_ws/src/rby1-sdk/models/rby1a/ur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
- link link_torso_4: geometry collision cylinder length=0.2 radius=0.105; visual mesh filename=file:///home/martin/umanoid_ws/src/rby1-sdk/models/rby1a/ur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
- link link_torso_5: geometry collision cylinder length=0.1350 radius=0.155; visual mesh filename=file:///home/martin/umanoid_ws/src/rby1-sdk/models/rby1a/ur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
- link wheel_l: geometry visual mesh filename=file:///home/martin/umanoid_ws/src/rby1-sdk/models/rby1a/ur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
- link wheel_r: geometry visual mesh filename=file:///home/martin/umanoid_ws/src/rby1-sdk/models/rby1a/ur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
Joints:
- joint left_wheel: limit velocity=15.707963268 -> effort=100.0 velocity=15.707963268
- joint right_wheel: limit velocity=15.707963268 -> effort=100.0 velocity=15.707963268
